File: autopilot_main_board.kicad_sch (KiCad schematic)
At the start: 4 parts

Commit message: Initial PCB layout
Parts:
- added FM1, FM2, FM3: ~, Fiducial:Fiducial_1mm_Mask2mm, symbol Mechanical:Fiducial
Other:
- sheet ESP32-C6 renamed ESP32
- sheet can renamed NMEA2000
- sheet external_connectors renamed Connectors
- note added: "Fiducial markers"
- note added: "Mounting holes M3"
- moved on the sheet: H1, H2, H3, H4
