File: current_sense_1.kicad_sch (KiCad schematic)
At the start: 7 parts

Commit message: Initial PCB layout
Other:
- moved on the sheet: R27
Changed lines of the file:
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@@
 	(wire
 		(pts
-			(xy 87.63 88.9) (xy 105.41 88.9)
+			(xy 87.63 88.9) (xy 104.14 88.9)
 		)
 		(stroke
@@
 	(wire
 		(pts
-			(xy 113.03 88.9) (xy 118.11 88.9)
+			(xy 111.76 88.9) (xy 118.11 88.9)
 		)
 		(stroke
@@
 	(symbol
 		(lib_id "Device:R")
-		(at 109.22 88.9 90)
+		(at 107.95 88.9 90)
 		(unit 1)
 		(exclude_from_sim no)
@@
 		(fields_autoplaced yes)
 		(property "Reference" "R27"
-			(at 109.22 82.55 90)
+			(at 107.95 82.55 90)
 			(effects
 				(font
@@
 		)
 		(property "Value" "1.5k"
-			(at 109.22 85.09 90)
+			(at 107.95 85.09 90)
 			(effects
 				(font
@@
 		)
 		(property "Footprint" "Resistor_SMD:R_0603_1608Metric"
-			(at 109.22 90.678 90)
+			(at 107.95 90.678 90)
 			(effects
 				(font
@@
 		)
 		(property "Datasheet" "~"
-			(at 109.22 88.9 0)
+			(at 107.95 88.9 0)
 			(effects
 				(font
@@
 		)
 		(property "Description" "Resistor"
-			(at 109.22 88.9 0)
-			(effects
-				(font
+			(at 107.95 88.9 0)
+			(effects
+				(font
