File: external_connectors.kicad_sch (KiCad schematic)
At the start: 23 parts, among them J1 Conn_01x05, J10 Screw_Terminal_01x02, J2 Conn_ARM_JTAG_SWD_10, J3 Conn_02x06_Top_Bottom, J4 Conn_01x04, J5 Screw_Terminal_01x03, J6 Conn_01x05_Pin, J8 Conn_01x02_Socket, J9 Conn_01x02_Socket

Commit message: Initial PCB layout
Connections:
- net EXT_PB10: now also J3.5 (Pin_5); no longer J3.2 (Pin_2)
- net EXT_PC13: now also J3.7 (Pin_7); no longer J3.4 (Pin_4)
- net EXT_PC14: now also J3.9 (Pin_9); no longer J3.5 (Pin_5)
- net EXT_PC15: now also J3.11 (Pin_11); no longer J3.6 (Pin_6)
- net GND: now also J3.2 (Pin_2), J3.4 (Pin_4), J3.6 (Pin_6); no longer J3.11 (Pin_11), J3.7 (Pin_7), J3.9 (Pin_9)
- net NMEA2000_GND: now also J6.5 (Pin_5); no longer J6.3 (Pin_3)
- net NMEA2000_H: now also J6.3 (Pin_3); no longer J6.4 (Pin_4)
- net NMEA2000_L: now also J6.4 (Pin_4); no longer J6.5 (Pin_5)
