File: stspin32g4.kicad_sch (KiCad schematic)
At the start: 38 parts, among them SW1 SW_Push_Open, U1 STSPIN32G4, Y1 24MHz

Commit message: Initial PCB layout
Parts:
- L1: footprint Inductor_SMD:L_0603_1608Metric -> Inductor_SMD:L_1206_3216Metric
Changed lines of the file:
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@@
 	(wire
 		(pts
-			(xy 165.1 104.14) (xy 184.15 104.14)
+			(xy 165.1 104.14) (xy 191.77 104.14)
 		)
 		(stroke
@@
 	(wire
 		(pts
+			(xy 168.91 101.6) (xy 165.1 101.6)
+		)
+		(stroke
+			(width 0)
+			(type default)
+		)
+	)
+	(wire
+		(pts
 			(xy 46.99 78.74) (xy 46.99 71.12)
 		)
@@
 	)
 	(label "SCREF"
-		(at 184.15 104.14 180)
+		(at 191.77 104.14 180)
 		(effects
 			(font
@@
 	(global_label "EXT_PD2"
 		(shape bidirectional)
-		(at 165.1 101.6 0)
+		(at 168.91 101.6 0)
 		(fields_autoplaced yes)
 		(effects
@@
 		)
 		(property "Intersheetrefs" "${INTERSHEET_REFS}"
-			(at 177.2397 101.6 0)
+			(at 181.0497 101.6 0)
 			(effects
 				(font
@@
 			)
 		)
-		(property "Footprint" "Inductor_SMD:L_0603_1608Metric"
+		(property "Footprint" "Inductor_SMD:L_1206_3216Metric"
 			(at 199.39 35.56 0)
 			(effects
