File: esp32.kicad_sch (KiCad schematic)
At the start: 3 parts, among them SW2 SW_Push_Open, U3 ESP32-C6-MINI-1

Commit message: Initial PCB layout
Parts:
- U3: footprint RF_Module:ESP32-C6-MINI-1 -> 1_SOC:ESP32-C6-MINI-1
Changed lines of the file:
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@@
 			)
 		)
-		(property "Footprint" "RF_Module:ESP32-C6-MINI-1"
+		(property "Footprint" "1_SOC:ESP32-C6-MINI-1"
 			(at 161.29 114.3 0)
 			(effects

Commit message: Continued routing
Parts:
- added C36: 10uF, Capacitor_SMD:C_1206_3216Metric, symbol Device:C
- added C37: 100nF, Capacitor_SMD:C_1206_3216Metric, symbol Device:C
Connections:
- net GND: now also C36.2, C37.2
- net VDD: now also C36.1, C37.1
